File: MIDI.kicad_pcb (KiCad board)
At the start: 2 copper layers, 59.2 x 48.8 mm, 26 parts, among them J1 MIDI IN, J2 MIDI OUT, J3 MIDI THRU, J4 DB25_Female, U1 6N136S, U2 MAX232, U3 L78L05

Commit message: Add files via upload
Parts:
- moved R6 3.56 mm to (146.8, 94.5)
Connections:
- D2 pad 1: GND -> Net-(D2-Pad1)
- D3 pad 1: GND -> Net-(D3-Pad1)
- R3 pad 1: Net-(R3-Pad1) -> Net-(D2-Pad1)
- R5 pad 1: Net-(R5-Pad1) -> Net-(D3-Pad1)
- R6 pad 1: Net-(R3-Pad1) -> +5V
- R8 pad 1: Net-(R7-Pad2) -> +5V
- U2 pad 12: Net-(R3-Pad1) -> Net-(D2-Pad1)
- U2 pad 9: Net-(R5-Pad1) -> Net-(D3-Pad1)
Routing:
- net Net-(D3-Pad1): track 0.00 -> 47.2 mm
- net Net-(R5-Pad1): track 28.0 -> 0.00 mm
- net Net-(D2-Pad1): track 0.00 -> 24.7 mm
- net Net-(R3-Pad1): track 24.5 -> 0.00 mm
- net Net-(R7-Pad2): track 41.7 -> 29.8 mm
- net +5V: track 81.5 -> 87.6 mm
- net Net-(D1-Pad1): track 21.0 -> 24.4 mm
- net Net-(D2-Pad2): track 7.57 -> 10.6 mm
- net Net-(J2-Pad5): track 9.25 -> 12.0 mm
- net Net-(J3-Pad5): track 9.25 -> 12.0 mm
- net Net-(J1-Pad5): track 9.25 -> 12.0 mm
- net Net-(J3-Pad4): track 9.19 -> 11.8 mm
- net Net-(J2-Pad4): track 9.19 -> 11.8 mm
- net /+12V: track 10.6 -> 12.6 mm
- net Net-(D3-Pad2): track 3.30 -> 2.59 mm
Other:
- board text added: "AMIGA SERIAL MIDI ADAPTER V1.1"
- board text removed: "AMIGA SERIAL MIDI ADAPTER V1.0"

Commit message: Update MIDI.kicad_pcb
Parts:
- J4: footprint Connector_Dsub:DSUB-25_Female_Horizontal_P2.77x2.84mm_EdgePinOffset4.94mm_Housed_MountingHolesOffset7.48mm -> Connector_Dsub:DSUB-25_Female_Horizontal_P2.77x2.84mm_EdgePinOffset7.70mm_Housed_MountingHolesOffset9.12mm
Other:
- board text added: "AMIGA SERIAL MIDI ADAPTER V1.2"
- board text removed: "AMIGA SERIAL MIDI ADAPTER V1.1"
Changed lines of the file:
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@@
     )
   )
-  (footprint "Connector_Dsub:DSUB-25_Female_Horizontal_P2.77x2.84mm_EdgePinOffset4.94mm_Housed_MountingHolesOffset7.48mm" (layer "F.Cu")
+  (footprint "Connector_Dsub:DSUB-25_Female_Horizontal_P2.77x2.84mm_EdgePinOffset7.70mm_Housed_MountingHolesOffset9.12mm" (layer "F.Cu")
     (at 131.069 81.834 180)
-    (descr "25-pin D-Sub connector, horizontal/angled (90 deg), THT-mount, female, pitch 2.77x2.84mm, pin-PCB-offset 4.9399999999999995mm, distance of mounting holes 47.1mm, distance of mounting holes to PCB edge 7.4799999999999995mm, see https://disti-assets.s3.amazonaws.com/tonar/files/datasheets/16730.pdf")
-    (tags "25-pin D-Sub connector horizontal angled 90deg THT female pitch 2.77x2.84mm pin-PCB-offset 4.9399999999999995mm mounting-holes-distance 47.1mm mounting-hole-offset 47.1mm")
-    (property "Sheetfile" "MIDI.kicad_sch")
-    (property "Sheetname" "")
-    (attr through_hole)
-    (fp_text reference "J4" (at 11.435 -3.51) (layer "F.SilkS")
-      (effects (font (size 1 1) (thickness 0.15)))
-    )
-    (fp_text value "DB25_Female" (at -16.62 15.85) (layer "F.Fab")
-      (effects (font (size 1 1) (thickness 0.15)))
-    )
-    (fp_line (start 0 -3.221325) (end -0.25 -3.654338) (layer "F.SilkS") (width 0.12))
-    (fp_line (start 0.25 -3.654338) (end 0 -3.221325) (layer "F.SilkS") (width 0.12))
-    (fp_line (start -43.23 7.72) (end -43.23 -2.76) (layer "F.SilkS") (width 0.12))
-    (fp_line (start -0.25 -3.654338) (end 0.25 -3.654338) (layer "F.SilkS") (width 0.12))
-    (fp_line (start -43.23 -2.76) (end 9.99 -2.76) (layer "F.SilkS") (width 0.12))
-    (fp_line (start 9.99 -2.76) (end 9.99 7.72) (layer "F.SilkS") (width 0.12))
-    (fp_line (start -43.7 -3.25) (end -43.7 14.85) (layer "F.CrtYd") (width 0.05))
-    (fp_line (start 10.45 14.85) (end 10.45 -3.25) (layer "F.CrtYd") (width 0.05))
-    (fp_line (start 10.45 -3.25) (end -43.7 -3.25) (layer "F.CrtYd") (width 0.05))
-    (fp_line (start -43.7 14.85) (end 10.45 14.85) (layer "F.CrtYd") (width 0.05))
-    (fp_line (start 8.53 7.78) (end 8.53 0.3) (layer "F.Fab") (width 0.1))
-    (fp_line (start 9.93 7.78) (end -43.17 7.78) (layer "F.Fab") (width 0.1))
-    (fp_line (start 9.93 -2.7) (end -43.17 -2.7) (layer "F.Fab") (width 0.1))
-    (fp_line (start 9.43 13.18) (end 9.43 8.18) (layer "F.Fab") (width 0.1))
-    (fp_line (start 9.93 7.78) (end 9.93 -2.7) (layer "F.Fab") (width 0.1))
-    (fp_line (start 9.43 8.18) (end 4.43 8.18) (layer "F.Fab") (width 0.1))
-    (fp_line (start 5.33 7.78) (end 5.33 0.3) (layer "F.Fab") (width 0.1))
-    (fp_line (start -43.17 7.78) (end -43.17 8.18) (layer "F.Fab") (width 0.1))
-    (fp_line (start -42.67 8.18) (end -42.67 13.18) (layer "F.Fab") (width 0.1))
-    (fp_line (start -37.67 8.18) (end -42.67 8.18) (layer "F.Fab") (width 0.1))
-    (fp_line (start 2.53 8.18) (end -35.77 8.18) (layer "F.Fab") (width 0.1))
-    (fp_line (start 9.93 8.18) (end 9.93 7.78) (layer "F.Fab") (width 0.1))
-    (fp_line (start -43.17 8.18) (end 9.93 8.18) (layer "F.Fab") (width 0.1))
-    (fp_line (start -38.57 7.78) (end -38.57 0.3) (layer "F.Fab") (width 0.1))
-    (fp_line (start -41.77 7.78) (end -41.77 0.3) (layer "F.Fab") (width 0.1))
-    (fp_line (start -42.67 13.18) (end -37.67 13.18) (layer "F.Fab") (width 0.1))
-    (fp_line (start -37.67 13.18) (end -37.67 8.18) (layer "F.Fab") (width 0.1))
-    (fp_line (start 2.53 14.35) (end 2.53 8.18) (layer "F.Fab") (width 0.1))
-    (fp_line (start -43.17 -2.7) (end -43.17 7.78) (layer "F.Fab") (width 0.1))
-    (fp_line (start -35.77 8.18) (end -35.77 14.35) (layer "F.Fab") (width 0.1))
-    (fp_line (start 4.43 8.18) (end 4.43 13.18) (layer "F.Fab") (width 0.1))
-    (fp_line (start 4.43 13.18) (end 9.43 13.18) (layer "F.Fab") (width 0.1))
-    (fp_line (start -35.77 14.35) (end 2.53 14.35) (layer "F.Fab") (width 0.1))
-    (fp_line (start -43.17 7.78) (end 9.93 7.78) (layer "F.Fab") (width 0.1))
-    (fp_arc (start -41.77 0.3) (mid -40.17 -1.3) (end -38.57 0.3) (layer "F.Fab") (width 0.1))
-    (fp_arc (start 5.33 0.3) (mid 6.93 -1.3) (end 8.53 0.3) (layer "F.Fab") (width 0.1))
-    (pad "0" thru_hole circle (at 6.93 0.3 180) (size 4 4) (drill 3.2) (layers *.Cu *.Mask)
+    (descr "25-pin D-Sub connector, horizontal/angled (90 deg), THT-mount, female, pitch 2.77x2.84mm, pin-PCB-offset 7.699999999999999mm, distance of mounting holes 47.1mm, distance of mounting holes to PCB edge 9.12mm, see https://disti-assets.s3.amazonaws.com/tonar/files/datasheets/16730.pdf")
+    (tags "25-pin D-Sub connector horizontal angled 90deg THT female pitch 2.77x2.84mm pin-PCB-offset 7.699999999999999mm mounting-holes-distance 47.1mm mounting-hole-offset 47.1mm")
+    (property "Sheetfile" "MIDI.kicad_sch")
+    (property "Sheetname" "")
+    (attr through_hole)
+    (fp_text reference "J4" (at -16.62 -2.8 180) (layer "F.SilkS")
+      (effects (font (size 1 1) (thickness 0.15)))
+    )
+    (fp_text value "DB25_Female" (at -16.62 18.61 180) (layer "F.Fab")
+      (effects (font (size 1 1) (thickness 0.15)))
+    )
+    (fp_text user "${REFERENCE}" (at -16.62 14.025 180) (layer "F.Fab")
+      (effects (font (size 1 1) (thickness 0.15)))
+    )
+    (fp_line (start -0.25 -2.754338) (end 0.25 -2.754338) (layer "F.SilkS") (width 0.12))
+    (fp_line (start 9.99 -1.86) (end 9.99 10.48) (layer "F.SilkS") (width 0.12))
+    (fp_line (start 0.25 -2.754338) (end 0 -2.321325) (layer "F.SilkS") (width 0.12))
+    (fp_line (start -43.23 10.48) (end -43.23 -1.86) (layer "F.SilkS") (width 0.12))
+    (fp_line (start 0 -2.321325) (end -0.25 -2.754338) (layer "F.SilkS") (width 0.12))
+    (fp_line (start -43.23 -1.86) (end 9.99 -1.86) (layer "F.SilkS") (width 0.12))
+    (fp_line (start 10.45 -2.35) (end -43.7 -2.35) (layer "F.CrtYd") (width 0.05))
+    (fp_line (start 10.45 17.65) (end 10.45 -2.35) (layer "F.CrtYd") (width 0.05))
+    (fp_line (start -43.7 17.65) (end 10.45 17.65) (layer "F.CrtYd") (width 0.05))
+    (fp_line (start -43.7 -2.35) (end -43.7 17.65) (layer "F.CrtYd") (width 0.05))
+    (fp_line (start -43.17 -1.8) (end -43.17 10.54) (layer "F.Fab") (width 0.1))
+    (fp_line (start 4.43 10.94) (end 4.43 15.94) (layer "F.Fab") (width 0.1))
+    (fp_line (start 5.33 10.54) (end 5.33 1.42) (layer "F.Fab") (width 0.1))
+    (fp_line (start -43.17 10.54) (end -43.17 10.94) (layer "F.Fab") (width 0.1))
+    (fp_line (start 9.93 10.54) (end -43.17 10.54) (layer "F.Fab") (width 0.1))
+    (fp_line (start 9.93 -1.8) (end -43.17 -1.8) (layer "F.Fab") (width 0.1))
+    (fp_line (start 9.93 10.54) (end 9.93 -1.8) (layer "F.Fab") (width 0.1))
+    (fp_line (start 8.53 10.54) (end 8.53 1.42) (layer "F.Fab") (width 0.1))
+    (fp_line (start -42.67 10.94) (end -42.67 15.94) (layer "F.Fab") (width 0.1))
+    (fp_line (start 9.93 10.94) (end 9.93 10.54) (layer "F.Fab") (width 0.1))
+    (fp_line (start -43.17 10.54) (end 9.93 10.54) (layer "F.Fab") (width 0.1))
+    (fp_line (start 4.43 15.94) (end 9.43 15.94) (layer "F.Fab") (width 0.1))
+    (fp_line (start -38.57 10.54) (end -38.57 1.42) (layer "F.Fab") (width 0.1))
+    (fp_line (start 2.53 10.94) (end -35.77 10.94) (layer "F.Fab") (width 0.1))
+    (fp_line (start -35.77 10.94) (end -35.77 17.11) (layer "F.Fab") (width 0.1))
+    (fp_line (start -37.67 15.94) (end -37.67 10.94) (layer "F.Fab") (width 0.1))
+    (fp_line (start -37.67 10.94) (end -42.67 10.94) (layer "F.Fab") (width 0.1))
+    (fp_line (start 2.53 17.11) (end 2.53 10.94) (layer "F.Fab") (width 0.1))
+    (fp_line (start 9.43 10.94) (end 4.43 10.94) (layer "F.Fab") (width 0.1))
+    (fp_line (start -35.77 17.11) (end 2.53 17.11) (layer "F.Fab") (width 0.1))
+    (fp_line (start -42.67 15.94) (end -37.67 15.94) (layer "F.Fab") (width 0.1))
+    (fp_line (start 9.43 15.94) (end 9.43 10.94) (layer "F.Fab") (width 0.1))
+    (fp_line (start -41.77 10.54) (end -41.77 1.42) (layer "F.Fab") (width 0.1))
+    (fp_line (start -43.17 10.94) (end 9.93 10.94) (layer "F.Fab") (width 0.1))
+    (fp_arc (start 5.33 1.42) (mid 6.93 -0.18) (end 8.53 1.42) (layer "F.Fab") (width 0.1))
+    (fp_arc (start -41.77 1.42) (mid -40.17 -0.18) (end -38.57 1.42) (layer "F.Fab") (width 0.1))
+    (pad "0" thru_hole circle (at -40.17 1.42 180) (size 4 4) (drill 3.2) (layers *.Cu *.Mask)
       (net 9 "GND"))
-    (pad "0" thru_hole circle (at -40.17 0.3 180) (size 4 4) (drill 3.2) (layers *.Cu *.Mask)
+    (pad "0" thru_hole circle (at 6.93 1.42 180) (size 4 4) (drill 3.2) (layers *.Cu *.Mask)
       (net 9 "GND"))
     (pad "1" thru_hole rect (at 0 0 180) (size 1.6 1.6) (drill 1) (layers *.Cu *.Mask)
@@
     (pad "25" thru_hole circle (at -31.855 2.84 180) (size 1.6 1.6) (drill 1) (layers *.Cu *.Mask)
       (net 27 "unconnected-(J4-Pad25)") (pinfunction "P25") (pintype "passive"))
-    (model "${KICAD6_3DMODEL_DIR}/Connector_Dsub.3dshapes/DSUB-25_Female_Horizontal_P2.77x2.84mm_EdgePinOffset4.94mm_Housed_MountingHolesOffset7.48mm.wrl"
+    (model "${KICAD6_3DMODEL_DIR}/Connector_Dsub.3dshapes/DSUB-25_Female_Horizontal_P2.77x2.84mm_EdgePinOffset7.70mm_Housed_MountingHolesOffset9.12mm.wrl"
       (offset (xyz 0 0 0))
       (scale (xyz 1 1 1))
@@
   )
   (gr_rect (start 177.292 75.946) (end 118.11 124.714) (layer "Edge.Cuts") (width 0.1) (fill none))
-  (gr_text "AMIGA SERIAL\nMIDI ADAPTER\nV1.1" (at 128.27 117.856) (layer "B.SilkS")
+  (gr_text "AMIGA SERIAL\nMIDI ADAPTER\nV1.2" (at 128.27 117.856) (layer "B.SilkS")
     (effects (font (size 1 1) (thickness 0.15)) (justify mirror))
   )
