File: MIDI.kicad_pcb (KiCad board)
At the start: 2 copper layers, 59.2 x 48.8 mm, 26 parts, among them J1 MIDI IN, J2 MIDI OUT, J3 MIDI THRU, J4 DB25_Female, U1 6N136S, U2 MAX232, U3 L78L05

Commit message: Add files via upload
Parts:
- removed G***: LOGO, Symbol:openhardware
- C1: value 100pF -> 0.1uF
- J4: footprint Connector_Dsub:DSUB-25_Female_Horizontal_P2.77x2.84mm_EdgePinOffset7.70mm_Housed_MountingHolesOffset9.12mm -> Connector_Dsub:DSUB-25_Female_Horizontal_P2.77x2.84mm_EdgePinOffset4.94mm_Housed_MountingHolesOffset7.48mm
- U3: value L78L05 -> UAL78L05ACLP; footprint Package_TO_SOT_THT:TO-220-3_Vertical -> Package_TO_SOT_THT:TO-92L_Inline
- moved D3 12.7 mm to (166.6, 99.3)
- moved R8 12.5 mm to (153.9, 99.3), turned to 0 degrees
- moved D2 4.14 mm to (146.7, 99.3)
- moved U3 2.94 mm to (150.7, 88.2), turned to 0 degrees
- moved R5 1.76 mm to (128.3, 102.8)
- moved C1 1.76 mm to (170.3, 102.8)
- moved R1 1.76 mm to (168.0, 102.8)
- moved R2 1.76 mm to (150.4, 102.8)
- moved R3 1.76 mm to (148.2, 102.8)
- moved R4 1.76 mm to (130.6, 102.8)
- moved C2 1.29 mm to (126.5, 98.1)
- moved C4 1.29 mm to (136.7, 98.1)
- moved C3 1.29 mm to (131.6, 98.1)
- moved C5 1.29 mm to (121.1, 90.0)
- moved U2 1.29 mm to (123.9, 95.1)
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Connections:
- J2 pad : GND -> (no net)
- J3 pad : GND -> (no net)
- J4 pad 0: GND -> (no net)
- U3 pad 1: /+12V -> +5V
- U3 pad 3: +5V -> /+12V
Routing:
- net Net-(D3-Pad1): track 47.2 -> 70.4 mm
- net +5V: track 87.6 -> 79.6 mm
- net Net-(D3-Pad2): track 2.59 -> 9.93 mm
- net Net-(J2-Pad5): track 12.0 -> 7.85 mm
- net Net-(J3-Pad5): track 12.0 -> 7.85 mm
- net Net-(J1-Pad5): track 12.0 -> 7.85 mm
- net Net-(D1-Pad1): track 24.4 -> 21.9 mm
- net Net-(D2-Pad2): track 10.6 -> 8.53 mm
- net /RXD: track 28.4 -> 26.4 mm
- net Net-(J3-Pad4): track 11.8 -> 10.2 mm
- net /+12V: track 12.6 -> 11.0 mm
- net Net-(R7-Pad2): track 29.8 -> 28.6 mm
- net Net-(C5-Pad2): track 7.55 -> 6.40 mm
- net Net-(D1-Pad2): track 18.8 -> 19.7 mm
- net Net-(J2-Pad4): track 11.8 -> 10.9 mm
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Other:
- board text added: "AMIGA SERIAL MIDI ADAPTER V1.3"
- board text added: "RX-IN"
- board text added: "TX-OUT"
- board text removed: "AMIGA SERIAL MIDI ADAPTER V1.2"

Commit message: Add files via upload
Parts:
- added REF**: OSHW-Logo_5.7x6mm_Copper, Symbol:OSHW-Logo_5.7x6mm_Copper, B.Cu at (147.8, 117.9)
- U3: value UAL78L05ACLP -> L4931-5.0
- moved U3 2.50 mm to (153.2, 88.2), turned to 180 degrees

Commit message: Add files via upload
Parts:
- added G***: LOGO, Symbol:RetronicDesign, B.Cu at (160.7, 116.4)
- added G***: LOGO, Symbol:MIDI, B.Cu at (127.8, 117.4)
- J4: footprint Connector_Dsub:DSUB-25_Female_Horizontal_P2.77x2.84mm_EdgePinOffset4.94mm_Housed_MountingHolesOffset7.48mm -> Connector_Dsub:DSUB-25_Female_Horizontal_P2.77x2.84mm_EdgePinOffset7.70mm_Housed_MountingHolesOffset9.12mm
- moved REF** 9.96 mm to (137.8, 117.4)
- moved U3 1.50 mm to (152.2, 87.0)
- moved C1 0.35 mm to (170.3, 102.5)
- moved R1 0.35 mm to (168.0, 102.5)
- moved R2 0.35 mm to (150.4, 102.5)
- moved R3 0.35 mm to (148.2, 102.5)
- moved R4 0.35 mm to (130.6, 102.5)
- moved R5 0.35 mm to (128.3, 102.5)
Connections:
- J4 pad 0: (no net) -> GND
Routing:
- net /+12V: track 11.0 -> 11.7 mm
- net Net-(J3-Pad4): track 10.2 -> 9.51 mm
- net Net-(D3-Pad1): track 70.4 -> 71.0 mm
Other:
- board text added: "AMIGA SERIAL ADAPTER V1.3"
- board text removed: "AMIGA SERIAL MIDI ADAPTER V1.3"
