File: MIDI.kicad_sch (KiCad schematic)
At the start: 25 parts, among them J1 MIDI IN, J2 MIDI OUT, J3 MIDI THRU, J4 DB25_Female, U1 6N136S, U2 MAX232, U3 L78L05

Commit message: Add files via upload
Connections:
- net +5V: now also R6.1, R8.1
- net GND: no longer D2.1 (K), D3.1 (K)
- net at R7.2, U1.6, U2.11 (T1IN): no longer R8.1
- net at R3.1, U2.12 (R1OUT): now also D2.1 (K); no longer R6.1
- net at R5.1, U2.9 (R2OUT): now also D3.1 (K)
Other:
- moved on the sheet: D2, D3, R6, R8

Commit message: Add files via upload
Parts:
- removed J1: MIDI IN, Downloads:MIDI_DIN5, symbol Connector:DIN-5
- removed J2: MIDI OUT, Downloads:MIDI_DIN5, symbol Connector:DIN-5
- removed J3: MIDI THRU, Downloads:MIDI_DIN5, symbol Connector:DIN-5
- added J1: MIDI IN, Downloads:MIDI_DIN5, symbol Connector:DIN-5_180degree
- added J?: MIDI OUT, Downloads:MIDI_DIN5, symbol Connector:DIN-5_180degree
- added J?: MIDI THRU, Downloads:MIDI_DIN5, symbol Connector:DIN-5_180degree
- C1: value 100pF -> 0.1uF
- U3: value L78L05 -> UAL78L05ACLP; footprint Package_TO_SOT_THT:TO-220-3_Vertical -> Package_TO_SOT_THT:TO-92L_Inline
Connections:
- net +12V: now also U3.3 (IN); no longer U3.1 (IN)
- net +5V: now also U3.1 (OUT); no longer U3.3 (OUT)
- net GND: now also J?.2, J?.2
- net at R1.2: now also J1.5
- net at D1.1 (K), U1.2: now also J1.4
- net at R2.2: now also J?.4
- net at R3.2: now also J?.5
- net at C1.1: now also J1.2
- net at R4.2: now also J?.4
- net at R5.2: now also J?.5
Other:
- moved on the sheet: C1

Commit message: Add files via upload
Parts:
- C1: value 0.1uF -> 100pF
- U3: value UAL78L05ACLP -> L4931-5.0
Other:
- note added: "POWER REGULATOR (250mA)"
- note removed: "POWER REGULATOR"
Changed lines of the file:
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@@
     (effects (font (size 1.27 1.27)) (justify left bottom))
   )
-  (text "POWER REGULATOR" (at 211.455 109.22 0)
-    (effects (font (size 1.27 1.27)) (justify left bottom))
+  (text "POWER REGULATOR\n(250mA)" (at 231.394 110.744 180)
+    (effects (font (size 1.27 1.27)) (justify right bottom))
   )
   (label "+12V" (at 241.3 118.745 0)
@@
     (in_bom yes) (on_board yes) (fields_autoplaced)
     (property "Reference" "U3" (id 0) (at 219.075 111.76 0))
-    (property "Value" "UAL78L05ACLP" (id 1) (at 219.075 114.3 0))
+    (property "Value" "L4931-5.0" (id 1) (at 219.075 114.3 0))
     (property "Footprint" "Package_TO_SOT_THT:TO-92L_Inline" (id 2) (at 219.075 113.665 0)
       (effects (font (size 1.27 1.27) italic) hide)
@@
   (symbol (lib_name "C_1") (lib_id "pspice:C") (at 28.5496 71.1708 0) (unit 1)
     (in_bom yes) (on_board yes) (fields_autoplaced)
-    (property "Reference" "C1" (id 0) (at 31.7246 69.9007 0)
-      (effects (font (size 1.27 1.27)) (justify left))
-    )
-    (property "Value" "0.1uF" (id 1) (at 31.7246 72.4407 0)
+    (property "Reference" "C1" (id 0) (at 31.75 69.9007 0)
+      (effects (font (size 1.27 1.27)) (justify left))
+    )
+    (property "Value" "100pF" (id 1) (at 31.75 72.4407 0)
       (effects (font (size 1.27 1.27)) (justify left))
     )
@@
     )
     (path "/884d8b47-767f-4aad-90d6-99332fce8e5a"
-      (reference "C1") (unit 1) (value "0.1uF") (footprint "Capacitor_THT:C_Disc_D3.0mm_W1.6mm_P2.50mm")
+      (reference "C1") (unit 1) (value "100pF") (footprint "Capacitor_THT:C_Disc_D3.0mm_W1.6mm_P2.50mm")
     )
     (path "/ac190baa-e212-49e4-9145-c81c3a965757"
@@
     )
     (path "/568e1785-f4d2-4fc6-9d89-77f57ec7e2c3"
-      (reference "U3") (unit 1) (value "UAL78L05ACLP") (footprint "Package_TO_SOT_THT:TO-92L_Inline")
-    )
-  )
+      (reference "U3") (unit 1) (value "L4931-5.0") (footprint "Package_TO_SOT_THT:TO-92L_Inline")
+    )
+  )

Commit message: Add files via upload
Parts:
- J4: footprint Connector_Dsub:DSUB-25_Female_Horizontal_P2.77x2.84mm_EdgePinOffset4.94mm_Housed_MountingHolesOffset7.48mm -> Connector_Dsub:DSUB-25_Female_Horizontal_P2.77x2.84mm_EdgePinOffset7.70mm_Housed_MountingHolesOffset9.12mm
Changed lines of the file:
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@@
       (effects (font (size 1.27 1.27)) (justify left))
     )
-    (property "Footprint" "Connector_Dsub:DSUB-25_Female_Horizontal_P2.77x2.84mm_EdgePinOffset4.94mm_Housed_MountingHolesOffset7.48mm" (id 2) (at 255.27 108.585 0)
+    (property "Footprint" "Connector_Dsub:DSUB-25_Female_Horizontal_P2.77x2.84mm_EdgePinOffset7.70mm_Housed_MountingHolesOffset9.12mm" (id 2) (at 255.27 108.585 0)
       (effects (font (size 1.27 1.27)) hide)
     )
@@
     )
     (path "/a2d52fd8-e19e-4876-89cd-8107fa438050"
-      (reference "J4") (unit 1) (value "DB25_Female") (footprint "Connector_Dsub:DSUB-25_Female_Horizontal_P2.77x2.84mm_EdgePinOffset4.94mm_Housed_MountingHolesOffset7.48mm")
+      (reference "J4") (unit 1) (value "DB25_Female") (footprint "Connector_Dsub:DSUB-25_Female_Horizontal_P2.77x2.84mm_EdgePinOffset7.70mm_Housed_MountingHolesOffset9.12mm")
     )
     (path "/b279a835-112a-490d-86a1-30b744210fbb"
